Commit message: Replace ROS 2 source workspace

File: src/ur5_sim_package/urdf/parallel_gripper.urdf.xacro (robot description, xacro)
@@ -104,10 +104,14 @@
         </material>
       </visual>
-      <collision>
-        <origin xyz="0 0 0" rpy="0 0 0"/>
-        <geometry>
-          <mesh
-            filename="package://ur5_sim_package/meshes/gripper/gripper_finger_assembly.STL"
-            scale="0.001 0.001 0.001"/>
+      <collision name="left_slider_collision">
+        <origin xyz="0.0157 -0.065 0.0075" rpy="0 0 0"/>
+        <geometry>
+          <box size="0.0306 0.080 0.015"/>
+        </geometry>
+      </collision>
+      <collision name="left_contact_pad">
+        <origin xyz="0.0414 -0.01275 0.0785" rpy="0 0 0"/>
+        <geometry>
+          <box size="0.025 0.0255 0.117"/>
         </geometry>
       </collision>
@@ -128,65 +132,5 @@
       <parent link="${prefix}gripper_base_link"/>
       <child link="${prefix}left_finger_link"/>
-      <!-- Original position of the supplied finger assembly -->
-      <origin
-        xyz="-0.00122 0.097 0.0686"
-        rpy="0 0 0"/>
-      <!-- Finger slides along its local positive Y-axis -->
-      <axis xyz="0 1 0"/>
-      <!-- Travel is in metres -->
-      <limit
-        lower="0.0"
-        upper="0.035"
-        effort="50.0"
-        velocity="0.08"/>
-      <dynamics
-        damping="2.0"
-        friction="0.2"/>
-    </joint>
-    <!-- ====================================================== -->
-    <!-- Right mirrored moving finger                           -->
-    <!-- ====================================================== -->
-    <link name="${prefix}right_finger_link">
-      <visual>
-        <origin xyz="0 0 0" rpy="0 0 0"/>
-        <geometry>
-          <!-- The same supplied finger STL is reused -->
-          <mesh
-            filename="package://ur5_sim_package/meshes/gripper/gripper_finger_assembly.STL"
-            scale="0.001 0.001 0.001"/>
-        </geometry>
-        <material name="${prefix}right_finger_material">
-          <color rgba="0.65 0.65 0.68 1.0"/>
-        </material>
-      </visual>
-      <collision>
-        <origin xyz="0 0 0" rpy="0 0 0"/>
-        <geometry>
-          <mesh
-            filename="package://ur5_sim_package/meshes/gripper/gripper_finger_assembly.STL"
-            scale="0.001 0.001 0.001"/>
-        </geometry>
-      </collision>
-      <inertial>
-        <origin xyz="0 0 0.065" rpy="0 0 0"/>
-        <mass value="0.20"/>
-        <inertia
-          ixx="0.00075"
-          ixy="0.0"
-          ixz="0.0"
-          iyy="0.00050"
-          iyz="0.0"
-          izz="0.00060"/>
-      </inertial>
-    </link>
-    <joint name="${prefix}right_finger_joint"
-           type="prismatic">
-      <parent link="${prefix}gripper_base_link"/>
-      <child link="${prefix}right_finger_link"/>
-      <!--Opposite side of the gripper, 180-degree Z rotation -->
-      <origin
-        xyz="0.08129 -0.097 0.0687"
-        rpy="0 0 3.14159265"/>
-      <!--right finger frame is rotated by 180 degrees-->
+      <origin xyz="-0.00125 0.025 0.0686" rpy="0 0 0"/>
       <axis xyz="0 1 0"/>
       <limit
@@ -198,5 +142,60 @@
         damping="2.0"
         friction="0.2"/>
-      <!--The right finger follows the left. Multiplier of +1 is used because the right joint frame rotated by 180 degrees.-->
+    </joint>
+    <!-- ====================================================== -->
+    <!-- Right mirrored moving finger                           -->
+    <!-- ====================================================== -->
+    <link name="${prefix}right_finger_link">
+      <visual>
+        <origin xyz="0 0 0" rpy="0 0 0"/>
+        <geometry>
+          <!-- The same supplied finger STL is reused -->
+          <mesh
+            filename="package://ur5_sim_package/meshes/gripper/gripper_finger_assembly.STL"
+            scale="0.001 0.001 0.001"/>
+        </geometry>
+        <material name="${prefix}right_finger_material">
+          <color rgba="0.65 0.65 0.68 1.0"/>
+        </material>
+      </visual>
+      <collision name="right_slider_collision">
+        <origin xyz="0.0157 -0.065 0.0075" rpy="0 0 0"/>
+        <geometry>
+          <box size="0.0306 0.080 0.015"/>
+        </geometry>
+      </collision>
+      <collision name="right_contact_pad">
+        <origin xyz="0.0414 -0.01275 0.0785" rpy="0 0 0"/>
+        <geometry>
+          <box size="0.025 0.0255 0.117"/>
+        </geometry>
+      </collision>
+      <inertial>
+        <origin xyz="0 0 0.065" rpy="0 0 0"/>
+        <mass value="0.20"/>
+        <inertia
+          ixx="0.00075"
+          ixy="0.0"
+          ixz="0.0"
+          iyy="0.00050"
+          iyz="0.0"
+          izz="0.00060"/>
+      </inertial>
+    </link>
+    <joint name="${prefix}right_finger_joint"
+           type="prismatic">
+      <parent link="${prefix}gripper_base_link"/>
+      <child link="${prefix}right_finger_link"/>
+      <origin xyz="0.08129 -0.025 0.0687" rpy="0 0 3.14159265"/>
+      <axis xyz="0 1 0"/>
+      <limit
+        lower="0.0"
+        upper="0.035"
+        effort="50.0"
+        velocity="0.08"/>
+      <dynamics
+        damping="2.0"
+        friction="0.2"/>
+      <!-- Mirror the left finger. -->
       <mimic
         joint="${prefix}left_finger_joint"
@@ -204,4 +203,15 @@
         offset="0.0"/>
     </joint>
+    <!-- Keep the fingers in place until the controller starts. -->
+    <gazebo reference="${prefix}left_finger_link">
+      <gravity>false</gravity>
+      <mu1>1.5</mu1>
+      <mu2>1.5</mu2>
+    </gazebo>
+    <gazebo reference="${prefix}right_finger_link">
+      <gravity>false</gravity>
+      <mu1>1.5</mu1>
+      <mu2>1.5</mu2>
+    </gazebo>
     <!-- ====================================================== -->
     <!-- End-effector tool-centre-point frame                    -->

File: src/ur5_sim_package/urdf/ur.urdf.xacro (robot description, xacro)
@@ -40,7 +40,7 @@
      sim_gazebo="true"
      >
-     <origin xyz="0 0 0" rpy="0 0 0" />          <!-- position robot in the world -->
+     <origin xyz="0.30 0.20 0" rpy="0 0 1.5708" />
    </xacro:ur_robot>
-   <!-- Create and attach the gripper -->
+   <!-- Gripper assembly. -->
    <xacro:parallel_gripper
      parent="$(arg tf_prefix)tool0"
@@ -49,4 +49,5 @@
      name="UR5System"
      tf_prefix="$(arg tf_prefix)"
-     controller_params_file="$(find ur5_sim_package)/config/controllers.yaml"/>
+     controller_params_file="$(find ur5_sim_package)/config/controllers.yaml"
+     gripper_initial_position="0.035"/>
 </robot>

File: src/ur5_sim_package/urdf/ur_control.xacro (robot description, xacro)
@@ -1,11 +1,4 @@
 <?xml version="1.0"?>
 <robot xmlns:xacro="http://wiki.ros.org/xacro">
-  <!--
-    Simulation control definitions for the custom UR5 and gripper.
-    The arm and gripper interfaces are kept in separate macros for clarity,
-    but are inserted into one ros2_control system. Gazebo therefore exposes
-    one controller manager containing arm_controller, gripper_controller, and
-    joint_state_broadcaster, matching config/controllers.yaml and MoveIt.
-  -->
   <xacro:include filename="$(find ur5_sim_package)/urdf/inc/ur_joint_control.xacro"/>
   <xacro:include filename="$(find ur5_sim_package)/urdf/inc/ur_sensors.xacro"/>
@@ -22,25 +15,24 @@
   <xacro:macro name="gripper_control" params="
     tf_prefix
-    initial_position:=0.01
+    initial_position:=0.035
     ">
     <joint name="${tf_prefix}left_finger_joint">
       <command_interface name="position"/>
+      <command_interface name="effort"/>
       <state_interface name="position">
-        <!-- Start clear of the inner hard stop. -->
+        <!-- Initial gripper position. -->
         <param name="initial_value">${initial_position}</param>
       </state_interface>
       <state_interface name="velocity"/>
+      <state_interface name="effort"/>
     </joint>
     <joint name="${tf_prefix}right_finger_joint">
-      <!--
-        The physical joint remains a mimic of the left finger. Both command
-        interfaces receive the same target to avoid Fortress's unstable,
-        hard-coded mimic velocity loop at this small scale.
-      -->
-      <command_interface name="position"/>
       <state_interface name="position">
         <param name="initial_value">${initial_position}</param>
       </state_interface>
       <state_interface name="velocity"/>
+      <state_interface name="effort"/>
+      <param name="mimic">${tf_prefix}left_finger_joint</param>
+      <param name="multiplier">1.0</param>
     </joint>
   </xacro:macro>
@@ -49,6 +41,6 @@
     tf_prefix
     controller_params_file
-    initial_positions:=${dict(shoulder_pan_joint=0.0,shoulder_lift_joint=-1.57,elbow_joint=0.0,wrist_1_joint=-1.57,wrist_2_joint=0.0,wrist_3_joint=0.0)}
-    gripper_initial_position:=0.01
+    initial_positions:=${dict(shoulder_pan_joint=0.0,shoulder_lift_joint=-1.2,elbow_joint=-1.0,wrist_1_joint=-1.2,wrist_2_joint=-1.0,wrist_3_joint=0.0)}
+    gripper_initial_position:=0.035
     ">
     <ros2_control name="${name}" type="system">

File: src/ur5_sim_package/urdf/ur_macro.xacro (robot description, xacro)
@@ -307,5 +307,5 @@
          <safety_controller soft_lower_limit="${shoulder_pan_lower_limit + safety_pos_margin}" soft_upper_limit="${shoulder_pan_upper_limit - safety_pos_margin}" k_position="${safety_k_position}" k_velocity="0.0"/>
       </xacro:if>
-      <dynamics damping="0" friction="0"/>
+    <dynamics damping="50.0" friction="1.0"/>
     </joint>
     <joint name="${tf_prefix}shoulder_lift_joint" type="revolute">
@@ -319,5 +319,5 @@
          <safety_controller soft_lower_limit="${shoulder_lift_lower_limit + safety_pos_margin}" soft_upper_limit="${shoulder_lift_upper_limit - safety_pos_margin}" k_position="${safety_k_position}" k_velocity="0.0"/>
       </xacro:if>
-      <dynamics damping="0" friction="0"/>
+    <dynamics damping="50.0" friction="1.0"/>
     </joint>
     <joint name="${tf_prefix}elbow_joint" type="revolute">
@@ -331,5 +331,5 @@
          <safety_controller soft_lower_limit="${elbow_joint_lower_limit + safety_pos_margin}" soft_upper_limit="${elbow_joint_upper_limit - safety_pos_margin}" k_position="${safety_k_position}" k_velocity="0.0"/>
       </xacro:if>
-      <dynamics damping="0" friction="0"/>
+    <dynamics damping="30.0" friction="0.5"/>
     </joint>
     <joint name="${tf_prefix}wrist_1_joint" type="revolute">
@@ -343,5 +343,5 @@
          <safety_controller soft_lower_limit="${wrist_1_lower_limit + safety_pos_margin}" soft_upper_limit="${wrist_1_upper_limit - safety_pos_margin}" k_position="${safety_k_position}" k_velocity="0.0"/>
       </xacro:if>
-      <dynamics damping="0" friction="0"/>
+    <dynamics damping="10.0" friction="0.2"/>
     </joint>
     <joint name="${tf_prefix}wrist_2_joint" type="revolute">
@@ -355,5 +355,5 @@
          <safety_controller soft_lower_limit="${wrist_2_lower_limit + safety_pos_margin}" soft_upper_limit="${wrist_2_upper_limit - safety_pos_margin}" k_position="${safety_k_position}" k_velocity="0.0"/>
       </xacro:if>
-      <dynamics damping="0" friction="0"/>
+    <dynamics damping="10.0" friction="0.2"/>
     </joint>
     <joint name="${tf_prefix}wrist_3_joint" type="${wrist_3_joint_type}">
@@ -375,5 +375,5 @@
         </xacro:if>
       </xacro:unless>
-      <dynamics damping="0" friction="0"/>
+    <dynamics damping="5.0" friction="0.02"/>
     </joint>
     <link name="${tf_prefix}ft_frame"/>
